File: pcb/board.brd (EAGLE design)
At the start: 100 x 80 mm, 24 parts, among them J1 USB-MICRO-AB, P2 PIN-F-2X25-DISC-P2, P8 PIN-M-2X23, P9 PIN-M-2X23

Commit message: Small improvement
Parts:
- moved R15 1.27 mm to (20.3, 59.7)
Routing:
- net SPI_MISO: track 53.1 -> 51.9 mm
- net N$3: track 8.45 -> 7.93 mm
- net GND: track 170.2 -> 169.7 mm
Changed lines of the file:
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@@
 <element name="R10" library="tb" package="0204/5" value="100" x="41.81" y="24.13" rot="R180"/>
 <element name="R12" library="tb" package="0204/5" value="100" x="24.13" y="24.13" rot="R180"/>
-<element name="R15" library="tb" package="0204/5" value="100" x="19.05" y="59.69" rot="R180"/>
+<element name="R15" library="tb" package="0204/5" value="100" x="20.32" y="59.69" rot="R180"/>
 <element name="J1" library="tb" package="USB-MICRO-AB" value="USB-MICRO-AB" x="11.43" y="29.21" rot="R270"/>
 <element name="R4" library="tb" package="0204/5" value="4k7" x="22.86" y="30.48" rot="R180"/>
@@
 <contactref element="P1" pad="38"/>
 <contactref element="R15" pad="1"/>
-<wire x1="22.86" y1="59.69" x2="22.86" y2="60.96" width="0.3048" layer="16"/>
-<wire x1="22.86" y1="60.96" x2="27.94" y2="66.04" width="0.3048" layer="16"/>
+<wire x1="24.13" y1="59.69" x2="24.13" y2="62.23" width="0.3048" layer="16"/>
+<wire x1="24.13" y1="62.23" x2="27.94" y2="66.04" width="0.3048" layer="16"/>
 </signal>
 <signal name="SPI_MOSI">
@@
 <contactref element="R15" pad="2"/>
 <contactref element="P9" pad="18"/>
-<wire x1="15.24" y1="59.69" x2="15.24" y2="63.5" width="0.3048" layer="1"/>
-<wire x1="15.24" y1="63.5" x2="60.96" y2="63.5" width="0.3048" layer="1"/>
+<wire x1="16.51" y1="59.69" x2="16.51" y2="63.5" width="0.3048" layer="1"/>
+<wire x1="16.51" y1="63.5" x2="60.96" y2="63.5" width="0.3048" layer="1"/>
 <wire x1="60.96" y1="63.5" x2="63.5" y2="60.96" width="0.3048" layer="1"/>
 </signal>
@@
 <wire x1="21.915" y1="44.296" x2="21.915" y2="49.205" width="0.3048" layer="1"/>
 <wire x1="21.915" y1="49.205" x2="21.59" y2="49.53" width="0.3048" layer="1"/>
-<wire x1="19.05" y1="27.94" x2="20.32" y2="27.94" width="0.3048" layer="16"/>
-<wire x1="20.32" y1="27.94" x2="20.32" y2="48.26" width="0.3048" layer="16"/>
-<wire x1="20.32" y1="48.26" x2="21.59" y2="49.53" width="0.3048" layer="16"/>
 <wire x1="21.25" y1="39.15" x2="21.25" y2="36.999" width="0.3048" layer="1"/>
 <wire x1="21.25" y1="36.999" x2="21.265" y2="36.984" width="0.3556" layer="1"/>
@@
 <wire x1="19.05" y1="27.94" x2="15.555" y2="27.94" width="0.3048" layer="1"/>
 <wire x1="15.555" y1="27.94" x2="15.555" y2="27.91" width="0.3048" layer="1"/>
-<wire x1="20.32" y1="27.94" x2="22.86" y2="27.94" width="0.3048" layer="16"/>
+<wire x1="19.05" y1="27.94" x2="21.59" y2="27.94" width="0.3048" layer="16"/>
+<wire x1="21.59" y1="27.94" x2="22.86" y2="27.94" width="0.3048" layer="16"/>
 <wire x1="22.86" y1="27.94" x2="24.13" y2="26.67" width="0.3048" layer="16"/>
 <wire x1="24.13" y1="26.67" x2="24.13" y2="11.43" width="0.3048" layer="16"/>
@@
 <wire x1="26.67" y1="8.89" x2="83.82" y2="8.89" width="0.3048" layer="16"/>
 <wire x1="76.2" y1="25.4" x2="76.2" y2="15.24" width="0.6096" layer="16"/>
+<wire x1="21.59" y1="49.53" x2="21.59" y2="27.94" width="0.4064" layer="16"/>
 </signal>
 <signal name="N$13">

Commit message: RC1
Parts:
- moved R9 3.81 mm to (34.3, 22.9)
- moved R2 3.81 mm to (55.9, 39.4)
- moved R3 3.81 mm to (59.7, 39.4)
- moved R10 1.27 mm to (41.8, 25.4)
Connections:
- net SAFE_L: now also P8.40; no longer P8.39
- net SAFE_R: now also P8.39; no longer P8.40
Routing:
- net ENC_X0: track 28.8 -> 11.2 mm
- net N$6: track 55.1 -> 49.2 mm
- net FAIL: track 33.7 -> 28.1 mm
- net N$25: track 12.5 -> 7.18 mm
- net ENC_X1: track 16.7 -> 22.0 mm
- net IRQ: track 31.7 -> 36.8 mm
- net SAFE_U: track 33.2 -> 28.6 mm
- net SAFE_L: track 34.0 -> 37.7 mm
- net SAFE_R: track 28.5 -> 32.2 mm
- net SPI_MOSI: track 45.9 -> 42.3 mm
- net SPI_MISO: track 51.9 -> 55.1 mm
- net UART2_RX: track 61.4 -> 58.2 mm
- net SAFE_B: track 28.5 -> 31.6 mm
- net N$19: track 42.7 -> 39.7 mm
- net HEAD_UP: track 30.7 -> 33.7 mm
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