File: pcb/board.sch (EAGLE design)
At the start: 24 parts, among them J1 USB-MICRO-AB, P1 PIN-F-2X25-DISC-P1, P2 PIN-F-2X25-DISC-P2, P8 PIN-M-2X23, P9 PIN-M-2X23

Commit message: RC1
Connections:
- net SAFE_L: now also P8.40; no longer P8.39
- net SAFE_R: now also P8.39; no longer P8.40
